File: pcb/kicad/wackymxter.kicad_sch (KiCad schematic)
At the start: 75 parts, among them J1 OLED_128x32, J2 Conn_01x03, U1 Pico, U3 TRRS

Commit message: [KiCAD] rev 0.3: dual diodes, optional hotswap
Parts:
- removed R1, R2: Resistor, Resistor_THT:R_Axial_DIN0204_L3.6mm_D1.6mm_P5.08mm_Horizontal, symbol ScottoKeebs:Placeholder_Resistor
- D1, D10, D11, D12, D13, D14, D15, D16, D17, D18, D19, D2, D20, D21, D22, D23, D24, D25, D26, D27, D28, D29, D3, D30, D31, D32, D33, D34, D4, D5, D6, D7, D8, D9: footprint ScottoKeebs_Components:Diode_DO-35 -> Keebio-Parts:Diode-dual
- S1, S10, S11, S12, S13, S14, S15, S16, S17, S18, S19, S2, S20, S21, S22, S23, S24, S25, S26, S27, S28, S29, S3, S30, S31, S32, S33, S34, S4, S5, S6, S7, S8, S9: footprint ScottoKeebs_MX:MX_PCB_1.00u -> keyswitches:Kailh_socket_MX_optional
Connections:
- net GND: now also U1.13 (GND)
- net LED1: now also U1.20 (GPIO15); no longer U1.29 (GPIO22)
- net RX0: now also U3.3 (RING1); no longer U3.4 (RING2)
- net SCL: now also U1.5 (GPIO3); no longer U1.7 (GPIO5)
- net SDA: now also U1.4 (GPIO2); no longer U1.6 (GPIO4)
- net TX0: now also U3.4 (RING2); no longer U3.3 (RING1)
- net VCC: no longer U3.2 (TIP)
- net col0: now also U1.25 (GPIO19); no longer U1.27 (GPIO21)
- net col2: now also U1.27 (GPIO21); no longer U1.25 (GPIO19)
- net col3: now also U1.9 (GPIO6); no longer U1.12 (GPIO9)
- net col4: now also U1.10 (GPIO7); no longer U1.11 (GPIO8)
- net col5: now also U1.11 (GPIO8); no longer U1.10 (GPIO7)
- net col6: now also U1.12 (GPIO9); no longer U1.9 (GPIO6)
- net VSYS: now reaches U1.39 (VSYS)
- net VSYS: now also U3.2 (TIP)
Other:
- title: (none) -> WackyMXter
- moved on the sheet: J1, J2, U3
