File: pcb-xiao/left/wackymxter_left.kicad_pcb (KiCad board)
At the start: 2 copper layers, 162.7 x 127 mm, 81 parts, among them U1 xiao-ble, U2 74HC595

Commit message: Insane progresgress
Parts:
- BATTCONN1: moved to B.Cu
- U1: footprint mcu:xiao-ble-smd-cutout -> wackymxter:xiao-ble-smd-cutout
- moved BATTCONN1 1.95 mm to (202.8, 71.9), turned to 180 degrees
Routing:
- net BATT: track 12.2 -> 15.1 mm
- net GND: track 109.0 -> 111.2 mm

Commit message: Cooler cutout out and match schematics
Parts:
- removed H8: MountingHole, MountingHole:MountingHole_2.2mm_M2
- moved H2 35.5 mm to (196.2, 124.7)
Other:
- board size 162.7 x 127 mm -> 162.7 x 131.6 mm
